Commit message: Added urdfs and rviz config

File: src/description/urdf/arena.urdf (robot description, URDF)
Before this commit: robot arena, 1 links, 0 joints
Links:
- link world: geometry visual mesh filename=package://description/meshes/arena.dae

Commit message: Changed base frame from world to map

File: src/description/urdf/arena.urdf (robot description, URDF)
Before this commit: robot arena, 1 links, 0 joints
Links:
- removed link world
- added link map; visual mesh filename=package://description/meshes/arena.dae
