Commit message: Started adding robot meshes

File: src/description/urdf/robot.urdf (robot description, URDF)
Before this commit: robot robot, 3 links, 2 joints
Links:
- removed link frame

Commit message: Placed central drive

File: src/description/urdf/robot.urdf (robot description, URDF)
Before this commit: robot robot, 2 links, 2 joints
Links:
- added link central_drive; visual mesh filename=package://description/meshes/central_drive.stl
Joints:
- added joint frame_to_central_drive: type fixed, parent frame, child central_drive, origin xyz=0.64135 -0.098425 0.022225 rpy=0 0 0

Commit message: Added bucket

File: src/description/urdf/robot.urdf (robot description, URDF)
Before this commit: robot robot, 3 links, 3 joints
Links:
- added link bucket; visual mesh filename=package://description/meshes/bucket.stl
Joints:
- added joint frame_to_bucket: type fixed, parent frame, child bucket, origin xyz=-0.2286 0.0 0.4318 rpy=0 0 0

Commit message: Fixed axes

File: src/description/urdf/robot.urdf (robot description, URDF)
Before this commit: robot robot, 4 links, 4 joints
Links:
- removed link sensor
Joints:
- removed joint frame_to_sensor
- joint frame_to_bucket: axis (none) -> 0 1 0; limit (none) -> lower=-3.14 upper=3.14 effort=1000.0 velocity=1000.0; type fixed -> revolute
- joint frame_to_central_drive: origin xyz=0.64135 -0.098425 0.022225 rpy=0 0 0 -> xyz=0.5291836 0.0 0.079375 rpy=0 0 0

Commit message: Placed monoboom

File: src/description/urdf/robot.urdf (robot description, URDF)
Before this commit: robot robot, 3 links, 3 joints
Links:
- added link monoboom; visual mesh filename=package://description/meshes/monoboom.stl
Joints:
- added joint central_drive_to_monoboom: type revolute, parent central_drive, child monoboom, origin xyz=0.0 0.0 0.0 rpy=0 -${pi/2} 0, axis 0 1 0, limit lower=-${pi} upper=0.0 effort=1000.0 velocity=1000.0

Commit message: Finished urdf

File: src/description/urdf/robot.urdf (robot description, URDF)
Before this commit: robot robot, 4 links, 4 joints
Links:
- added link backhoe_bucket; visual mesh filename=package://description/meshes/backhoe_bucket.stl
Joints:
- added joint monoboom_to_backhoe_bucket: type revolute, parent monoboom, child backhoe_bucket, origin xyz=0.55245 0.0 0.0 rpy=0 -${pi/2} 0, axis 0 1 0, limit lower=-${pi} upper=${pi} effort=1000.0 velocity=1000.0

Commit message: Close enough

File: src/description/urdf/robot.urdf (robot description, URDF)
Before this commit: robot robot, 5 links, 5 joints
Joints:
- joint central_drive_to_monoboom: limit lower=-${pi} upper=0.0 effort=1000.0 velocity=1000.0 -> lower=0.0 upper=3.0 effort=1000.0 velocity=1000.0; origin xyz=0.0 0.0 0.0 rpy=0 -${pi/2} 0 -> xyz=0.0 0.0 0.0 rpy=0 ${pi/2} 0
- joint frame_to_bucket: limit lower=-3.14 upper=3.14 effort=1000.0 velocity=1000.0 -> lower=${-2*pi} upper=${2*pi} effort=1000.0 velocity=1000.0; origin xyz=-0.2286 0.0 0.4318 rpy=0 0 0 -> xyz=-0.2286 0.0 0.4318 rpy=0 -${80/180*pi} 0
- joint monoboom_to_backhoe_bucket: limit lower=-${pi} upper=${pi} effort=1000.0 velocity=1000.0 -> lower=-1.32 upper=2.0 effort=1000.0 velocity=1000.0

Commit message: Received correct mapping from Josh

File: src/description/urdf/robot.urdf (robot description, URDF)
Before this commit: robot robot, 5 links, 5 joints
Joints:
- joint central_drive_to_monoboom: limit lower=0.0 upper=3.0 effort=1000.0 velocity=1000.0 -> lower=0.0 upper=3.14 effort=1000.0 velocity=1000.0
- joint frame_to_bucket: origin xyz=-0.2286 0.0 0.4318 rpy=0 -${80/180*pi} 0 -> xyz=-0.2286 0.0 0.4318 rpy=0 -${85/180*pi} 0

Commit message: Added servos to urdf

File: src/description/urdf/robot.urdf (robot description, URDF)
Before this commit: robot robot, 5 links, 5 joints
Links:
- added link left_dynamixel; visual mesh filename=package://description/meshes/left_dynamixel.stl
- added link right_dynamixel; visual mesh filename=package://description/meshes/right_dynamixel.stl
Joints:
- added joint frame_to_left_dynamixel: type fixed, parent frame, child left_dynamixel, origin xyz=-0.186436 0.3137916 0.3756406 rpy=0 0 0
- added joint frame_to_right_dynamixel: type fixed, parent frame, child right_dynamixel, origin xyz=-0.186436 -0.3137916 0.3756406 rpy=0 0 0

Commit message: Added camera mount to urdf

File: src/description/urdf/robot.urdf (robot description, URDF)
Before this commit: robot robot, 7 links, 7 joints
Links:
- added link left_camera_mount; visual mesh filename=package://description/meshes/camera_mount.stl
- added link right_camera_mount; visual mesh filename=package://description/meshes/camera_mount.stl
Joints:
- added joint left_dynamixel_to_camera_mount: type fixed, parent left_dynamixel, child left_camera_mount, origin xyz=0.000508 0.016256 0.0195072 rpy=0 0 0
- added joint right_dynamixel_to_camera_mount: type fixed, parent right_dynamixel, child right_camera_mount, origin xyz=0.000508 -0.016256 0.0195072 rpy=0 0 ${pi}

Commit message: Added camera to urdf

File: src/description/urdf/robot.urdf (robot description, URDF)
Before this commit: robot robot, 9 links, 9 joints
Links:
- removed link left_camera_mount
- removed link left_dynamixel
- removed link right_camera_mount
- removed link right_dynamixel
Joints:
- removed joint frame_to_left_dynamixel
- removed joint frame_to_right_dynamixel
- removed joint left_dynamixel_to_camera_mount
- removed joint right_dynamixel_to_camera_mount

Commit message: Added mapping from linear actuator to backhoe curl

File: src/description/urdf/robot.urdf (robot description, URDF)
Before this commit: robot robot, 5 links, 5 joints
Links:
- added link monoboom_actuator_link
Joints:
- added joint monoboom_actuator: type prismatic, parent monoboom, child monoboom_actuator_link, origin xyz=0.1 0.0 0.0 rpy=0 0 0, axis 1 0 0, limit lower=0 upper=0.1778 effort=1000.0 velocity=1000.0
- joint monoboom_to_backhoe_bucket: limit lower=-1.32 upper=2.0 effort=1000.0 velocity=1000.0 -> lower=-10 upper=10.0 effort=1000.0 velocity=1000.0; origin xyz=0.55245 0.0 0.0 rpy=0 -${pi/2} 0 -> xyz=0.55245 0.0 0.0 rpy=0 ${5*pi/8} ${pi}

Commit message: added rotation and offset to urdf

File: src/description/urdf/robot.urdf (robot description, URDF)
Before this commit: robot robot, 6 links, 6 joints
Links:
- added link imu
Joints:
- added joint imu_to_baselink: type fixed, parent base_link, child imu, origin xyz=.54 -.15 0.0 rpy=0 ${-pi/2} ${pi}

Commit message: updated imu transformation

File: src/description/urdf/robot.urdf (robot description, URDF)
Before this commit: robot robot, 7 links, 7 joints
Joints:
- joint imu_to_baselink: origin xyz=.54 -.15 0.0 rpy=0 ${-pi/2} ${pi} -> xyz=.54 -.15 0.0 rpy=${-pi/2} ${-pi/2} 0

Commit message: Added boxes

File: src/description/urdf/robot.urdf (robot description, URDF)
Before this commit: robot robot, 7 links, 7 joints
Links:
- added link battery_box; visual mesh filename=package://description/meshes/box.stl
- added link computer_box; visual mesh filename=package://description/meshes/box.stl
Joints:
- added joint frame_to_battery_box: type fixed, parent frame, child battery_box, origin xyz=0.858774 0.093726 0.132461 rpy=${pi/2} 0 0
- added joint frame_to_computer_box: type fixed, parent frame, child computer_box, origin xyz=0.858774 -0.093726 0.132461 rpy=${pi/2} 0 0

Commit message: Added zr300 servo

File: src/description/urdf/robot.urdf (robot description, URDF)
Before this commit: robot robot, 9 links, 9 joints
Links:
- added link zr300_dynamixel; visual mesh filename=package://description/meshes/zr300_dynamixel.stl
Joints:
- added joint computer_box_to_zr300_dynamixel: type fixed, parent computer_box, child zr300_dynamixel, origin xyz=0.0450596 0.0436118 0.0316484 rpy=0 0 0
- joint frame_to_battery_box: origin xyz=0.858774 0.093726 0.132461 rpy=${pi/2} 0 0 -> xyz=0.858774 0.093726 0.132461 rpy=0 0 0
- joint frame_to_computer_box: origin xyz=0.858774 -0.093726 0.132461 rpy=${pi/2} 0 0 -> xyz=0.858774 -0.093726 0.132461 rpy=0 0 0

Commit message: Added zr300 mount

File: src/description/urdf/robot.urdf (robot description, URDF)
Before this commit: robot robot, 10 links, 10 joints
Links:
- added link zr300_mount; visual mesh filename=package://description/meshes/zr300_mount.stl
Joints:
- added joint zr300_dynamixel_to_zr300_mount: type revolute, parent zr300_dynamixel, child zr300_mount, origin xyz=0.016256 0 0.0322072 rpy=0 0 0, axis 0 0 1, limit lower=${-pi} upper=${pi} effort=1000.0 velocity=1000.0

Commit message: Finished adding zr300

File: src/description/urdf/robot.urdf (robot description, URDF)
Before this commit: robot robot, 11 links, 11 joints
Links:
- added link zr300_mount_2; visual mesh filename=package://description/meshes/zr300_mount_2.stl
Joints:
- added joint zr300_mount_to_zr300_mount_2: type fixed, parent zr300_mount, child zr300_mount_2, origin xyz=0 0 0 rpy=0 0 0

Commit message: Fixed base_link

File: src/description/urdf/robot.urdf (robot description, URDF)
Before this commit: robot robot, 12 links, 12 joints
Links:
- added link frame; visual mesh filename=package://description/meshes/frame.stl
Joints:
- joint base_link_to_frame: origin xyz=0 0 2.0796e-01 rpy=0 0 0 -> xyz=-387.35e-3 0 2.0796e-01 rpy=0 0 0

Commit message: Fixed imu position and orientation

File: src/description/urdf/robot.urdf (robot description, URDF)
Before this commit: robot robot, 13 links, 12 joints
Joints:
- joint imu_to_baselink: origin xyz=.54 -.15 0.0 rpy=${-pi/2} ${-pi/2} 0 -> xyz=937.5e-3 -140.65e-3 105e-3 rpy=${-pi/2} 0 ${pi/2}; parent base_link -> frame

Commit message: added bumping to wc speeds and corrected imu in urdf

File: src/description/urdf/robot.urdf (robot description, URDF)
Before this commit: robot robot, 13 links, 12 joints
Joints:
- joint imu_to_baselink: origin xyz=937.5e-3 -140.65e-3 105e-3 rpy=${-pi/2} 0 ${pi/2} -> xyz=937.5e-3 -140.65e-3 105e-3 rpy=-1.52 0 ${-pi/2}

Commit message: updated the imu test

File: src/description/urdf/robot.urdf (robot description, URDF)
Before this commit: robot robot, 13 links, 12 joints
Links:
- added link imu_trans
Joints:
- added joint imu_to_imu_trans: type fixed, parent imu_trans, child imu, origin xyz=0 0 0 rpy=0 0 0
- joint imu_to_baselink: child imu -> imu_trans; origin xyz=937.5e-3 -140.65e-3 105e-3 rpy=-1.52 0 ${-pi/2} -> xyz=937.5e-3 -140.65e-3 105e-3 rpy=0 0 0

Commit message: Added orientation

File: src/description/urdf/robot.urdf (robot description, URDF)
Before this commit: robot robot, 14 links, 13 joints
Links:
- removed link imu_trans
Joints:
- removed joint imu_to_baselink
- removed joint imu_to_imu_trans
- added joint frame_to_imu: type fixed, parent frame, child imu, origin xyz=937.5e-3 -140.65e-3 105e-3 rpy=${-pi/2} 0 ${pi/2}
